Commit message: Updated description, added zed launch and bagging launch

File: defense_description/urdf/iiwa.urdf.xacro (robot description, xacro)
@@ -3,4 +3,5 @@
   <xacro:include filename="$(find iiwa_description)/urdf/materials.xacro" />
   <xacro:include filename="$(find iiwa_description)/urdf/iiwa7.xacro"/>
+  <xacro:include filename="$(find zed_wrapper)/urdf/zed_descr.urdf.xacro"/>
   <xacro:arg name="hardware_interface" default="PositionJointInterface"/>
   <xacro:arg name="robot_name" default="iiwa"/>
@@ -61,3 +62,8 @@
     <origin xyz="-0.01768 0.00131 0.20735" rpy="0 2.87979 0"/>
   </joint>
+  <joint name="zed_joint" type="fixed">
+    <parent link="world" />
+    <child link="zed_link" />
+    <origin xyz="-0.45 0 1.3716" rpy="0 0.523599 0"/>
+  </joint>
 </robot>

Commit message: Seems like it should work, with some adjustment to frames and spacing

File: defense_description/urdf/iiwa.urdf.xacro (robot description, xacro)
@@ -56,10 +56,4 @@
     <origin xyz="0 0 0" rpy="0 0 0"/>
   </joint>
-  <link name="tweeze_tips" />
-  <joint name="tweeze_joint" type="fixed">
-    <parent link="grip_link" />
-    <child link="tweeze_tips" />
-    <origin xyz="-0.01768 0.00131 0.20735" rpy="0 2.87979 0"/>
-  </joint>
   <joint name="zed_joint" type="fixed">
     <parent link="world" />
@@ -67,3 +61,9 @@
     <origin xyz="-0.45 0 1.3716" rpy="0 0.523599 0"/>
   </joint>
+  <link name="just_the_tip" />
+  <joint name="tip_joint" type="fixed">
+    <parent link="iiwa_link_ee" />
+    <child link="just_the_tip" />
+    <origin xyz="0 0 0" rpy="0 0 0"/>
+  </joint>
 </robot>

Commit message: Updated viz

File: defense_description/urdf/iiwa.urdf.xacro (robot description, xacro)
@@ -44,20 +44,8 @@
     <child link="env_link" />
   </joint>
-  <link name="grip_link">
-    <visual>
-      <geometry>
-        <mesh filename="package://defense_description/meshes/HandESmall.dae" />
-      </geometry>
-    </visual>
-  </link>
-  <joint name="grip_joint" type="fixed">
-    <parent link="iiwa_link_ee" />
-    <child link="grip_link" />
-    <origin xyz="0 0 0" rpy="0 0 0"/>
-  </joint>
   <joint name="zed_joint" type="fixed">
     <parent link="world" />
     <child link="zed_link" />
-    <origin xyz="-0.45 0 1.3716" rpy="0 0.523599 0"/>
+    <origin xyz="-0.4826 -0.2 1.3716" rpy="0 0.523599 0"/>
   </joint>
   <link name="just_the_tip" />
@@ -65,5 +53,5 @@
     <parent link="iiwa_link_ee" />
     <child link="just_the_tip" />
-    <origin xyz="0 0 0" rpy="0 0 0"/>
+    <origin xyz="0 0 0.2" rpy="0 3.14159 0"/>
   </joint>
 </robot>

Commit message: Updated urdf

File: defense_description/urdf/iiwa.urdf.xacro (robot description, xacro)
@@ -47,5 +47,5 @@
     <parent link="world" />
     <child link="zed_link" />
-    <origin xyz="-0.4826 -0.2 1.3716" rpy="0 0.523599 0"/>
+    <origin xyz="0.1524 -0.3616 -0.06985" rpy="0 0 0"/>
   </joint>
   <link name="just_the_tip" />
@@ -53,5 +53,11 @@
     <parent link="iiwa_link_ee" />
     <child link="just_the_tip" />
-    <origin xyz="0 0 0.2" rpy="0 3.14159 0"/>
+    <origin xyz="-0.04 -0.1 0.02" rpy="0 3.14159 -0.349"/>
+  </joint>
+  <link name="spray_origin_link" />
+  <joint name="spray_origin_joint" type="fixed">
+    <parent link="iiwa_link_0" />
+    <child link="spray_origin_link" />
+    <origin xyz="0 0 0.340" rpy="0 0 0"/>
   </joint>
 </robot>
